Commit message: Fixing Humanbot urdf Moving human legs back out of camera view and making camera invusuble

File: jarves_description/robots/kobuki_human_asus_xtion_pro.urdf.xacro (robot description, xacro)
@@ -2,12 +2,13 @@
 <!--
     - Base      : kobuki
-    - Stacks    : hexagons
-    - 3d Sensor : kinect
+    - Stacks    : human
+    - 3d Sensor : asus_xtion_pro_invisible
 -->
 <robot name="humanbot" xmlns:xacro="http://ros.org/wiki/xacro">
   <xacro:include filename="$(find turtlebot_description)/urdf/turtlebot_library.urdf.xacro" />
-  <xacro:include filename="$(find jarves_description)/robots/includes/person_standing.xacro" />
+  <xacro:include filename="$(find jarves_description)/urdf/sensors/asus_xtion_pro_invisible.urdf.xacro" />
+  <xacro:include filename="$(find jarves_description)/urdf/humans/person_standing.xacro" />
   <kobuki/>
-  <sensor_asus_xtion_pro          parent="base_link"/>
-  <person_standing                parent="base_link"/>
+  <sensor_asus_xtion_pro_invisible  parent="base_link"/>
+  <person_standing                  parent="base_link"/>
 </robot>

File: jarves_description/urdf/humans/person_standing.xacro (robot description, xacro)
@@ -5,5 +5,5 @@
   <xacro:macro name="person_standing" params="parent">
     <joint name="person_standing_joint" type="fixed">
-      <origin xyz="0.0 0.0 0.0" rpy="0 0 ${M_PI/2}"/>
+      <origin xyz="-0.1 0.0 0.0" rpy="0 0 ${M_PI/2}"/>
       <parent link="${parent}"/>
       <child link="person_standing_link"/>
