Commit message: Switching to person models in package

File: jarves_description/urdf/humans/person_standing.xacro (robot description, xacro)
@@ -13,5 +13,5 @@
         <origin xyz="0 0 0" rpy="0 0 0"/>
         <geometry>
-          <mesh filename="model://person_standing/meshes/standing.dae"/>
+          <mesh filename="package://jarves_description/meshes/humans/person_standing/meshes/standing.dae"/>
         </geometry>
       </visual>
